Commit message: obstacle viz, compute_spheres in Robot

File: assets/panda/panda_collision_spheres.urdf (robot description, URDF)
Before this commit: robot panda, 14 links, 13 joints
Joints:
- removed joint right_gripper
- added joint right_gripper_joint: type fixed, parent panda_link8, child right_gripper, origin xyz=0 0 0.1 rpy=0 0 2.35619449019, axis 0 0 1

File: assets/panda/panda_collision_spheres_gltf.urdf (robot description, URDF)
Before this commit: robot panda, 14 links, 13 joints
Joints:
- removed joint right_gripper
- added joint right_gripper_joint: type fixed, parent panda_link8, child right_gripper, origin xyz=0 0 0.1 rpy=0 0 2.35619449019, axis 0 0 1

File: assets/panda/panda_self_collision_spheres.urdf (robot description, URDF)
Before this commit: robot panda, 14 links, 13 joints
Joints:
- removed joint right_gripper
- added joint right_gripper_joint: type fixed, parent panda_link8, child right_gripper, origin xyz=0 0 0.1 rpy=0 0 2.35619449019, axis 0 0 1
